Commit message: finished rev1 of IVK

File: app/backend/python code/Sims/ROBOT.urdf (robot description, URDF)
Before this commit: robot robot, 8 links, 7 joints
Links:
- removed link bace_link
- added link base_link; collision cylinder length=0.186275 radius=0.05080; visual cylinder length=0.186275 radius=0.05080
- added link elbow_revolute_to_wrist_link; collision cylinder length=0.110 radius=0.05080; visual cylinder length=0.110 radius=0.05080
- added link sholder_to_elbow_link; collision cylinder length=0.114 radius=0.05080; visual cylinder length=0.114 radius=0.05080
Joints:
- added joint elbow_revolute_to_wrist_joint: type fixed, parent elbow_revolute_link, child elbow_revolute_to_wrist_link, origin xyz=0.0 0.0 0.212 rpy=-1.570796 0.0 0.0
- added joint sholder_to_elbow_joint: type fixed, parent sholder_link, child sholder_to_elbow_link, origin xyz=0.0 0.0 0.525 rpy=-1.570796 0.0 0.0
- joint bace_joint: child bace_link -> base_link; origin xyz=0.0 0.0 0.054725 rpy=0.0 0.0 0.0 -> xyz=0.0 0.0 0.054725 rpy=0.0 0.0 -1.570796
- joint elbow_joint: axis -1.0 0.0 0.0 -> 0.0 1.0 0.0; origin xyz=-0.114 0.0 0.525 rpy=3.141692 0.0 0.0 -> xyz=0.0 0.0 -0.114 rpy=-1.570796 0.0 0.0; parent sholder_link -> sholder_to_elbow_link
- joint elbow_revolute_joint: axis 0.0 0.0 1.0 -> 0.0 0.0 -1.0; limit lower=-3.141692 upper=3.141692 effort=60.0 velocity=100.0 -> lower=-1.570796 upper=1.570796 effort=60.0 velocity=100.0
- joint sholder_joint: axis 1.0 0.0 0.0 -> 0.0 1.0 0.0; limit lower=-3.141692 upper=3.141692 effort=60.0 velocity=100.0 -> lower=-1.570796 upper=1.570796 effort=60.0 velocity=100.0; parent bace_link -> base_link
- joint wrist_joint: axis 1.0 0.0 0.0 -> 0.0 -1.0 0.0; origin xyz=-0.110 0.0 0.212 rpy=3.141692 0.0 0.0 -> xyz=0.0 0.0 0.110 rpy=-1.570796 0.0 0.0; parent elbow_revolute_link -> elbow_revolute_to_wrist_link
