Commit message: fixing urdf and main bace joint not working

File: app/backend/python code/ROBOT.urdf (robot description, URDF)
Before this commit: robot robot, 10 links, 9 joints
Joints:
- removed joint bace_joint
- added joint base_joint: type revolute, parent table_link, child base_link, origin xyz=0.0 0.0 0.054725 rpy=0.0 0.0 0.0, axis 0.0 0.0 1.0, limit lower=-3.141692 upper=3.141692 effort=60.0 velocity=100.0
- joint table_joint: axis (none) -> 0 0 1; type fixed -> revolute

Commit message: finished FK sim for test IK algorithum

File: app/backend/python code/ROBOT.urdf (robot description, URDF)
Before this commit: robot robot, 10 links, 9 joints
Links:
- removed link world
- added link world_link; visual box size=0.0 0.0 0.0
Joints:
- joint base_joint: axis 0.0 0.0 1.0 -> 0 0 1
- joint elbow_joint: axis 0.0 1.0 0.0 -> 0 1 0
- joint elbow_revolute_joint: axis 0.0 0.0 -1.0 -> 0 0 -1
- joint sholder_joint: axis 0.0 1.0 0.0 -> 0 1 0
- joint table_joint: limit (none) -> lower=-3.14159265359 upper=3.14159265359 effort=100.0 velocity=3.0; parent world -> world_link
- joint wrist_joint: axis 0.0 -1.0 0.0 -> 0 -1 0
- joint wrist_revolute_link: axis 0.0 0.0 1.0 -> 0 0 1
