Commit message: fixed over rotashion in path for better move efficiently

File: app/backend/python code/urdf_tes1.urdf (robot description, URDF)
Before this commit: robot robot_arm, 9 links, 8 joints
Joints:
- joint shoulder_joint: limit lower=-1.57 upper=1.57 -> lower=-3.141592654 upper=3.141592654
