Commit message: found best work surface aria for robot and added error for IK and FK

File: app/backend/python code/urdf_tes2.urdf (robot description, URDF)
Before this commit: robot robot_arm, 9 links, 8 joints
Joints:
- joint elbow_joint: limit lower=-2.487094189 upper=2.487094189 effort=60.0 velocity=100.0 -> lower=-3.141692 upper=3.141692 effort=60.0 velocity=100.0

Commit message: ended up doing a lot of bug fixed and not much work on upgrading the DB

File: app/backend/python code/urdf_tes2.urdf (robot description, URDF)
Before this commit: robot robot_arm, 9 links, 8 joints
Joints:
- joint base_joint: axis 0 0 -1 -> 0 0 1; limit (none) -> lower=-6.283919 upper=6.283919; origin xyz=0 0 0.14735 rpy=0 0 0 -> xyz=0 0 0.14735 rpy=0 0 1.570796
- joint elbow_revolute_joint: axis 0 0 -1 -> 0 0 1
- joint wrist_joint: axis 0 -1 0 -> 0 1 0; limit lower=-3.141692 upper=3.141692 effort=60.0 velocity=100.0 -> lower=-3.141692 upper=3.141692

Commit message: protortype joint interpolated moshion and IMU controll

File: app/backend/python code/urdf_tes2.urdf (robot description, URDF)
Before this commit: robot robot_arm, 9 links, 8 joints
Joints:
- joint wrist_revolute_link: limit lower=-3.141692 upper=3.141692 effort=60.0 velocity=100.0 -> lower=-314.1692 upper=314.1692 effort=60.0 velocity=100.0

Commit message: finished joint intorpolashion program

File: app/backend/python code/urdf_tes2.urdf (robot description, URDF)
Before this commit: robot robot_arm, 9 links, 8 joints
Joints:
- joint elbow_joint: axis 0 1 0 -> 0 -1 0
